File: eagle/pcb/incubator.brd (EAGLE design)
At the start: 99.1 x 63.5 mm, 57 parts, among them IC1 MCP1703-50, J2 RJ12RIGHTANGLE-I2C, J7 22--02, Q1 BSP75, Q5 BSP75, X2 8MHz, X4 MINI-USB

Commit message: version 1.1
Parts:
- U$1: value EC11E -> ROTARYENCODER; device lpatiny:EC11E -> RotaryEncoder:ROTARYENCODER
- moved CX4 13.3 mm to (66.7, 22.9), turned to 90 degrees
- moved U$1 7.65 mm to (74.9, 14.6), turned to 0 degrees
Routing:
- net +12V: track 255.9 -> 250.8 mm
- net RX: track 68.9 -> 72.6 mm
- net GND: track 116.7 -> 114.7 mm, vias 17 -> 18
- net TX: track 65.0 -> 66.6 mm

Commit message: version 1.1.0
Connections:
- net A3: no longer R2.1
- net A4: no longer R1.1
- net A6: now also U$11.4
- net D11*: now also R1.1; no longer R6.3
- net D12*: now also U$11.6; no longer U$11.4
- net D6*: now also R2.1; no longer U$11.6
- net VCC: now also R6.3
Routing:
- net D11*: track 82.8 -> 23.9 mm
- net VCC: track 219.9 -> 238.8 mm
- net A6: track 0.00 -> 17.7 mm
- net A4: track 9.98 -> 0.00 mm
- net A3: track 9.76 -> 0.00 mm
- net D6*: track 16.6 -> 25.0 mm, vias 0 -> 2
- net D12*: track 20.8 -> 14.3 mm
- net TX: track 66.6 -> 65.8 mm
- net RX: track 72.6 -> 71.8 mm
- net XTAL1: track 16.1 -> 15.4 mm
Other:
- board text added: "Incubator v1.1.0"
- board text removed: "Incubator v1.0.0"
